File: pcbs/common/left.kicad_sch (KiCad schematic)
At the start: 87 parts, among them J1 ST-0277D00-052-142, J2 Conn_01x03, J3 TYPE-C-31-M-13C, SW1 SW_Push, SW10 SW_Push, SW11 SW_Push, SW12 SW_Push, SW13 SW_Push, SW14 SW_Push, SW15 SW_Push, SW16 SW_Push, SW17 SW_Push, SW18 SW_Push, SW19 SW_Push, SW2 SW_Push, SW20 SW_Push, SW21 SW_Push, SW22 SW_Push, SW23 SW_Push, SW24 SW_Push, SW3 SW_Push, SW4 SW_Push, SW5 SW_Push, SW6 SW_Push, SW7 SW_Push, SW8 SW_Push, SW9 SW_Push, U1 NCP1117LPST33T3G, U2 TPD4E05U06DQAR, U3 W25Q128JVSIQ, U4 RP2040, Y1 12MHz 18pF

Commit message: Add buildguide
Parts:
- added D2, D3: 1.5KExxA, Diode_THT:D_DO-201AE_P15.24mm_Horizontal, symbol Diode:1.5KExxA
- added Q1, Q2: NMOS, symbol Simulation_SPICE:NMOS
- added R10, R8: R, symbol Device:R
Connections:
- net GND: now also R10.2, R8.2
- new net: D2.2 (A2), R8.1
- new net: D3.2 (A2), R10.1
